Commit message: link sensors back to base_link

File: rover/src/kipp_description/urdf/kipp.urdf.xacro (robot description, xacro)
@@ -163,6 +163,6 @@
     <!-- ZED Localization -> The reference link is '$(arg camera_name)_camera_link' and 'base_link' is a child -->
     <joint name="$(arg camera_name)_joint" type="fixed">
-      <parent link="$(arg camera_name)_camera_link"/>
-      <child link="base_link"/>
+      <parent link="base_link"/>
+      <child link="$(arg camera_name)_camera_link"/>
       <origin
         xyz="-0.12 0.0 -0.25"

Commit message: partially done URDF

File: rover/src/kipp_description/urdf/kipp.urdf.xacro (robot description, xacro)
@@ -2,72 +2,67 @@
 <robot xmlns:xacro="http://www.ros.org/wiki/xacro" name="kipp">
 <xacro:include filename="$(find zed_wrapper)/urdf/zed_macro.urdf.xacro"/>
+<!-- Robot constants-->
+<xacro:property name="base_width" value = ""/>
+<xacro:property name="base_height" value = ""/>
+<xacro:property name="base_length" value = ""/>
+<xacro:property name="steering_xy" value=""/>
+<xacro:property name="steering_z" value=""/>
+<xacro:property name="wheel_radius" value = ""/>
+<xacro:property name="camera_y" value = ""/>
+<xacro:property name="camera_z" value = ""/>
+<xacro:propery name="gnss_x" value=""/>
+<xacro:propery name="gnss_y" value=""/>
+<xacro:propery name="gnss_z" value=""/>
+<xacro:propery name="footprint" value="${-((base_height/2)+wheel_radius)}"/>
+    <!-- Robot Base -->
    <link name="base_link">
         <visual>
-            <origin xyz="0.0 0.0 0.0" rpy="0.0 0.0 0.0"/>
             <geometry>
-                <box size= "0.8 0.5 0.5"/>
+                <box size="${base_length} ${base_width} ${base_height}"/>
             </geometry>
+            <material name="rover_material">
+                <color rgba="0.5 0.5 0.5 1.0" />
+            </material>
         </visual>
-   </link>
-   <link name="front_left_steering">
-        <visual>
-            <origin xyz="0.0 0.0 0.0" rpy="0.0 0.0 0.0"/>
-            <geometry>
-                <box size="0.1 0.1 0.1"/>
-            </geometry>
-        </visual>
-   </link>
-   <link name="front_right_steering">
-        <visual>
-            <origin xyz="0.0 0.0 0.0" rpy="0.0 0.0 0.0"/>
-            <geometry>
-                <box size="0.1 0.1 0.1"/>
-            </geometry>
-        </visual>
-   </link>
-   <link name="back_left_steering">
-        <visual>
-            <origin xyz="0.0 0.0 0.0" rpy="0.0 0.0 0.0"/>
-            <geometry>
-                <box size="0.1 0.1 0.1"/>
-            </geometry>
-        </visual>
-   </link>
-   <link name="back_right_steering">
-        <visual>
-            <origin xyz="0.0 0.0 0.0" rpy="0.0 0.0 0.0"/>
-            <geometry>
-                <box size="0.1 0.1 0.1"/>
-            </geometry>
-        </visual>
-   </link>
-   <joint name="front_left_steering_joint" type="revolute">
-    <parent link="base_link"/>
-    <child link="front_left_steering"/>
-    <axis xyz="0 0 1"/>
-    <origin xyz="0.4 0.25 -0.25" rpy="0 0 0"/>
-    <limit lower="-1.57" upper="1.57" effort="0.0" velocity="0.0"/>
-   </joint>
-   <joint name="front_right_steering_joint" type="revolute">
-    <parent link="base_link"/>
-    <child link="front_right_steering"/>
-    <axis xyz="0 0 1"/>
-    <origin xyz="0.4 -0.25 -0.25" rpy="0 0 0"/>
-    <limit lower="-1.57" upper="1.57" effort="0.0" velocity="0.0"/>
-   </joint>
-   <joint name="back_left_steering_joint" type="revolute">
-    <parent link="base_link"/>
-    <child link="back_left_steering"/>
-    <axis xyz="0 0 1"/>
-    <origin xyz="-0.4 0.25 -0.25" rpy="0 0 0"/>
-    <limit lower="-1.57" upper="1.57" effort="0.0" velocity="0.0"/>
-   </joint>
-   <joint name="back_right_steering_joint" type="revolute">
-    <parent link="base_link"/>
-    <child link="back_right_steering"/>
-    <axis xyz="0 0 1"/>
-    <origin xyz="-0.4 -0.25 -0.25" rpy="0 0 0"/>
-    <limit lower="-1.57" upper="1.57" effort="0.0" velocity="0.0"/>
-   </joint>
+    </link>
+    <!-- Robot Footprint -->
+    <link name="base_footprint"/>
+    <joint name="base_joint" type="fixed">
+        <parent link="base_link"/>
+        <child link="base_footprint"/>
+        <origin xyz="0.0 0.0 ${footprint}" rpy="0 0 0"/>
+    </joint>
+    <!-- Steering -->
+    <xacro:macro name="steering" params="prefix x_reflect y_reflect">
+        <link name="${prefix}_steering_link">
+            <visual>
+                <origin xyz="0 0 0" rpy="0 0 0"/>
+                <geometry>
+                    <box size="${steering_xy} ${steering_xy} ${steering_z}"/>
+                </geometry>
+                <material name="Gray">
+                    <color rgba="0.5 0.5 0.5 1.0"/>
+                </material>
+            </visual>
+        </link>
+        <joint name="${prefix}_steering_joint" type="revolute">
+            <parent link="base_link"/>
+            <child link="${prefix}_steering_link"/>
+            <axis xyz="0 0 1"/>
+            <origin xyz="${(x_reflect*base_length)/2} ${(y_reflect*base_width)/2} ${footprint+wheel_radius}" rpy="0 0 0"/>
+        </joint>
+    </xacro:macro>
+    <xacro:steering prefix="front_left" x_reflect="1" y_reflect="1"/>
+    <xacro:steering prefix="front_right" x_reflect="1" y_reflect="-1"/>
+    <xacro:steering prefix="back_left" x_reflect="-1" y_reflect="1"/>
+    <xacro:steering prefix="front_right" x_reflect="-1" y_reflect="-1"/>
+<!-- I GOT TO HERE - - - - - - - - - - - - - - - - - - - - - - - - - - - - - - - - - - - - - - - - - - - - -  - - -->
+<!-- I GOT TO HERE - - - - - - - - - - - - - - - - - - - - - - - - - - - - - - - - - - - - - - - - - - - - -  - - -->
+<!-- I GOT TO HERE - - - - - - - - - - - - - - - - - - - - - - - - - - - - - - - - - - - - - - - - - - - - -  - - -->
+<!-- I GOT TO HERE - - - - - - - - - - - - - - - - - - - - - - - - - - - - - - - - - - - - - - - - - - - - -  - - -->
+<!-- I GOT TO HERE - - - - - - - - - - - - - - - - - - - - - - - - - - - - - - - - - - - - - - - - - - - - -  - - -->
+<!-- I GOT TO HERE - - - - - - - - - - - - - - - - - - - - - - - - - - - - - - - - - - - - - - - - - - - - -  - - -->
+<!-- I GOT TO HERE - - - - - - - - - - - - - - - - - - - - - - - - - - - - - - - - - - - - - - - - - - - - -  - - -->
+<!-- I GOT TO HERE - - - - - - - - - - - - - - - - - - - - - - - - - - - - - - - - - - - - - - - - - - - - -  - - -->
     <link name="front_left_wheel">
         <visual>

Commit message: Cleaned up code and changed hardcoded vals w defined vars

File: rover/src/kipp_description/urdf/kipp.urdf.xacro (robot description, xacro)
@@ -121,43 +121,38 @@
     </joint>
    <!--Camera Addtion-->
-   <xacro:arg name="camera_name"   default="zed2i" />
-  <xacro:arg name="camera_model"  default="zed2i" />
-  <xacro:arg name="use_zed_localization" default="true" />
+    <xacro:arg name="camera_name"   default="zed2i" />
+    <xacro:arg name="camera_model"  default="zed2i" />
+    <xacro:arg name="use_zed_localization" default="true" />
     <xacro:zed_camera name="$(arg camera_name)" model="$(arg camera_model)" />
      <!-- Add the first ZED Camera -->
-      <xacro:if value="$(arg use_zed_localization)">
-    <!-- ZED Localization -> The reference link is '$(arg camera_name)_camera_link' and 'base_link' is a child -->
-    <joint name="$(arg camera_name)_joint" type="fixed">
-      <parent link="base_link"/>
-      <child link="$(arg camera_name)_camera_link"/>
-      <origin
-        xyz="-0.12 0.0 -0.25"
-        rpy="0 0 0"
-      />
-    </joint>
-  </xacro:if>
-  <xacro:unless value="$(arg use_zed_localization)">
-    <!-- NO ZED Localization -> '$(arg camera_name)_camera_link' is a child of 'base_link' -->
-    <joint name="$(arg camera_name)_joint" type="fixed">
-      <parent link="base_link"/>
-      <child link="$(arg camera_name)_camera_link"/>
-      <origin
-        xyz="0.12 0.0 0.25"
-        rpy="0 0 0"
-      />
-    </joint>
-  </xacro:unless>
-  <link name="gnss_link">
-        <visual>
-            <origin xyz="0.0 0.0 0.0" rpy="1.57 0.0 0.0"/>
-            <geometry>
-                <cylinder radius="0.05" length="0.05"/>
-            </geometry>
-        </visual>
-   </link>
-    <joint name="gnss_joint" type="fixed">
+    <xacro:if value="$(arg use_zed_localization)">
+        <!-- ZED Localization -> The reference link is '$(arg camera_name)_camera_link' and 'base_link' is a child -->
+        <joint name="$(arg camera_name)_joint" type="fixed">
         <parent link="base_link"/>
-        <child link="gnss_link"/>
-        <origin xyz="0 0 0.70" rpy="0 0 0"/>
-    </joint>
+        <child link="$(arg camera_name)_camera_link"/>
+        <origin xyz="${camera_y} ${camera_z}" rpy="0 0 0"/>
+        </joint>
+    </xacro:if>
+    <xacro:unless value="$(arg use_zed_localization)">
+        <!-- NO ZED Localization -> '$(arg camera_name)_camera_link' is a child of 'base_link' -->
+        <joint name="$(arg camera_name)_joint" type="fixed">
+        <parent link="base_link"/>
+        <child link="$(arg camera_name)_camera_link"/>
+        <origin xyz="${camera_y} ${camera_z}" rpy="0 0 0"/>
+        </joint>
+    </xacro:unless>
+<!--GNSS-->
+    <link name="gnss_link">
+            <visual>
+                <origin xyz="0.0 0.0 0.0" rpy="1.57 0.0 0.0"/>
+                <geometry>
+                    <cylinder radius="0.05" length="0.05"/> <!-- GNSS radius?-->
+                </geometry>
+            </visual>
+    </link>
+        <joint name="gnss_joint" type="fixed">
+            <parent link="base_link"/>
+            <child link="gnss_link"/>
+            <origin xyz="${gnss_x} ${gnss_y} ${gnss_z}" rpy="0 0 0"/> <!-- GNSS position -->
+        </joint>
 </robot>

Commit message: URDF done except sensors

File: rover/src/kipp_description/urdf/kipp.urdf.xacro (robot description, xacro)
@@ -3,16 +3,18 @@
 <xacro:include filename="$(find zed_wrapper)/urdf/zed_macro.urdf.xacro"/>
 <!-- Robot constants-->
-<xacro:property name="base_width" value = ""/>
-<xacro:property name="base_height" value = ""/>
-<xacro:property name="base_length" value = ""/>
-<xacro:property name="steering_xy" value=""/>
-<xacro:property name="steering_z" value=""/>
-<xacro:property name="wheel_radius" value = ""/>
-<xacro:property name="camera_y" value = ""/>
-<xacro:property name="camera_z" value = ""/>
-<xacro:propery name="gnss_x" value=""/>
-<xacro:propery name="gnss_y" value=""/>
-<xacro:propery name="gnss_z" value=""/>
-<xacro:propery name="footprint" value="${-((base_height/2)+wheel_radius)}"/>
+<xacro:property name="base_width" value= "0.5084"/>
+<xacro:property name="base_height" value="0.51"/>
+<xacro:property name="base_length" value="0.77975"/>
+<xacro:property name="steering_xy" value="0.06155"/>
+<xacro:property name="steering_z" value="0.23"/>
+<xacro:property name="wheel_radius" value="0.0909"/>
+<xacro:property name="wheel_width" value="0.1016"/>
+<xacro:property name="camera_y" value=""/>
+<xacro:property name="camera_z" value=""/>
+<xacro:property name="gnss_x" value=""/>
+<xacro:property name="gnss_y" value=""/>
+<xacro:property name="gnss_z" value=""/>
+<xacro:property name="PI" value="3.1415692"/>
+<xacro:property name="footprint" value="${-((base_height/2)+(wheel_radius))}"/>
     <!-- Robot Base -->
    <link name="base_link">
@@ -31,5 +33,5 @@
         <parent link="base_link"/>
         <child link="base_footprint"/>
-        <origin xyz="0.0 0.0 ${footprint}" rpy="0 0 0"/>
+        <origin xyz="0.0 0.0 ${footprint-wheel_radius}" rpy="0 0 0"/>
     </joint>
     <!-- Steering -->
@@ -50,5 +52,6 @@
             <child link="${prefix}_steering_link"/>
             <axis xyz="0 0 1"/>
-            <origin xyz="${(x_reflect*base_length)/2} ${(y_reflect*base_width)/2} ${footprint+wheel_radius}" rpy="0 0 0"/>
+            <origin xyz="${(x_reflect*base_length)/2} ${(y_reflect*base_width)/2} ${(footprint+wheel_radius)}" rpy="0 0 0"/>
+            <limit lower="${-(PI/2)}" upper="${(PI/2)}" effort="0.0" velocity="0.0"/>
         </joint>
     </xacro:macro>
@@ -56,96 +59,64 @@
     <xacro:steering prefix="front_right" x_reflect="1" y_reflect="-1"/>
     <xacro:steering prefix="back_left" x_reflect="-1" y_reflect="1"/>
-    <xacro:steering prefix="front_right" x_reflect="-1" y_reflect="-1"/>
-<!-- I GOT TO HERE - - - - - - - - - - - - - - - - - - - - - - - - - - - - - - - - - - - - - - - - - - - - -  - - -->
-<!-- I GOT TO HERE - - - - - - - - - - - - - - - - - - - - - - - - - - - - - - - - - - - - - - - - - - - - -  - - -->
-<!-- I GOT TO HERE - - - - - - - - - - - - - - - - - - - - - - - - - - - - - - - - - - - - - - - - - - - - -  - - -->
-<!-- I GOT TO HERE - - - - - - - - - - - - - - - - - - - - - - - - - - - - - - - - - - - - - - - - - - - - -  - - -->
-<!-- I GOT TO HERE - - - - - - - - - - - - - - - - - - - - - - - - - - - - - - - - - - - - - - - - - - - - -  - - -->
-<!-- I GOT TO HERE - - - - - - - - - - - - - - - - - - - - - - - - - - - - - - - - - - - - - - - - - - - - -  - - -->
-<!-- I GOT TO HERE - - - - - - - - - - - - - - - - - - - - - - - - - - - - - - - - - - - - - - - - - - - - -  - - -->
-<!-- I GOT TO HERE - - - - - - - - - - - - - - - - - - - - - - - - - - - - - - - - - - - - - - - - - - - - -  - - -->
-    <link name="front_left_wheel">
+    <xacro:steering prefix="back_right" x_reflect="-1" y_reflect="-1"/>
+    <!-- Edge Wheels -->
+    <xacro:macro name="edge_wheel" params="prefix x_reflect y_reflect">
+        <link name="${prefix}_wheel_link">
+            <visual>
+                <origin xyz="0 0 0" rpy="${PI/2} 0 0"/>
+                <geometry>
+                    <cylinder radius="${wheel_radius}" length="${wheel_width}"/>
+                </geometry>
+                <material name="black">
+                    <color rgba="0.0 0.0 0.0 1.0"/>
+                </material>
+            </visual>
+        </link>
+        <joint name="${prefix}_wheel_joint" type="continuous">
+            <parent link="base_link"/>
+            <child link="${prefix}_wheel_link"/>
+            <origin xyz="${(x_reflect*base_length)/2} ${(y_reflect*base_width)/2} ${footprint}" rpy="0 0 0"/>
+            <axis xyz="0 0 1"/>
+        </joint>
+    </xacro:macro>
+    <xacro:edge_wheel prefix="front_left" x_reflect="1" y_reflect="1"/>
+    <xacro:edge_wheel prefix="front_right" x_reflect="1" y_reflect="-1"/>
+    <xacro:edge_wheel prefix="back_left" x_reflect="-1" y_reflect="1"/>
+    <xacro:edge_wheel prefix="back_right" x_reflect="-1" y_reflect="-1"/>
+    <!-- Middle Left Wheel -->
+    <link name="middle_left_wheel_link">
         <visual>
-            <origin xyz="0.0 0.0 0.0" rpy="1.57 0.0 0.0"/>
+            <origin xyz="0 0 0" rpy="${PI/2} 0 0"/>
             <geometry>
-                <cylinder radius="0.1" length="0.05"/>
+                <cylinder radius="${wheel_radius}" length="${wheel_width}"/>
             </geometry>
+            <material name="black">
+                <color rgba="0.0 0.0 0.0 1.0"/>
+            </material>
         </visual>
-   </link>
-       <link name="front_right_wheel">
-        <visual>
-            <origin xyz="0.0 0.0 0.0" rpy="1.57 0.0 0.0"/>
-            <geometry>
-                <cylinder radius="0.1" length="0.05"/>
-            </geometry>
-        </visual>
-   </link>
-       <link name="middle_left_wheel">
-        <visual>
-            <origin xyz="0.0 0.0 0.0" rpy="1.57 0.0 0.0"/>
-            <geometry>
-                <cylinder radius="0.1" length="0.05"/>
-            </geometry>
-        </visual>
-   </link>
-       <link name="middle_right_wheel">
-        <visual>
-            <origin xyz="0.0 0.0 0.0" rpy="1.57 0.0 0.0"/>
-            <geometry>
-                <cylinder radius="0.1" length="0.05"/>
-            </geometry>
-        </visual>
-   </link>
-       <link name="back_left_wheel">
-        <visual>
-            <origin xyz="0.0 0.0 0.0" rpy="1.57 0.0 0.0"/>
-            <geometry>
-                <cylinder radius="0.1" length="0.05"/>
-            </geometry>
-        </visual>
-   </link>
-       <link name="back_right_wheel">
-        <visual>
-            <origin xyz="0.0 0.0 0.0" rpy="1.57 0.0 0.0"/>
-            <geometry>
-                <cylinder radius="0.1" length="0.05"/>
-            </geometry>
-        </visual>
-   </link>
-    <joint name="front_left_wheel_joint" type="continuous">
-        <parent link="front_left_steering"/>
-        <child link="front_left_wheel"/>
-        <axis xyz="0 0 1"/>
-        <origin xyz="0 0 0" rpy="0 0 0"/>
-    </joint>
-    <joint name="front_right_wheel_joint" type="continuous">
-        <parent link="front_right_steering"/>
-        <child link="front_right_wheel"/>
-        <axis xyz="0 0 1"/>
-        <origin xyz="0 0 0" rpy="0 0 0"/>
-    </joint>
+    </link>
     <joint name="middle_left_wheel_joint" type="continuous">
         <parent link="base_link"/>
-        <child link="middle_left_wheel"/>
+        <child link="middle_left_wheel_link"/>
+        <origin xyz="0 ${(base_width)/2} ${footprint}" rpy="0 0 0"/>
         <axis xyz="0 0 1"/>
-        <origin xyz="0 -0.25 -0.25" rpy="0 0 0"/>
     </joint>
-    <joint name="middle_right_wheel_joint_" type="continuous">
+    <!-- Middle Right Wheel -->
+    <link name="middle_right_wheel_link">
+        <visual>
+            <origin xyz="0 0 0" rpy="${PI/2} 0 0"/>
+            <geometry>
+                <cylinder radius="${wheel_radius}" length="${wheel_width}"/>
+            </geometry>
+            <material name="black">
+                <color rgba="0.0 0.0 0.0 1.0"/>
+            </material>
+        </visual>
+    </link>
+    <joint name="middle_right_wheel_joint" type="continuous">
         <parent link="base_link"/>
-        <child link="middle_right_wheel"/>
+        <child link="middle_right_wheel_link"/>
+        <origin xyz="0 ${-(base_width)/2} ${footprint}" rpy="0 0 0"/>
         <axis xyz="0 0 1"/>
-        <origin xyz="0 0.25 -0.25" rpy="0 0 0"/>
-    </joint>
-    <joint name="back_left_wheel_joint" type="continuous">
-        <parent link="back_left_steering"/>
-        <child link="back_left_wheel"/>
-        <axis xyz="0 0 1"/>
-        <origin xyz="0 0 0" rpy="0 0 0"/>
-    </joint>
-    <joint name="back_right_wheel_joint" type="continuous">
-        <parent link="back_right_steering"/>
-        <child link="back_right_wheel"/>
-        <axis xyz="0 0 1"/>
-        <origin xyz="0 0 0" rpy="0 0 0"/>
     </joint>
    <!--Camera Addtion-->

Commit message: update urdf

File: rover/src/kipp_description/urdf/kipp.urdf.xacro (robot description, xacro)
@@ -100,5 +100,5 @@
         <child link="middle_left_wheel_link"/>
         <origin xyz="0 ${(base_width)/2} ${footprint}" rpy="0 0 0"/>
-        <axis xyz="0 0 1"/>
+        <axis xyz="0 1 0"/>
     </joint>
     <!-- Middle Right Wheel -->
@@ -118,5 +118,5 @@
         <child link="middle_right_wheel_link"/>
         <origin xyz="0 ${-(base_width)/2} ${footprint}" rpy="0 0 0"/>
-        <axis xyz="0 0 1"/>
+        <axis xyz="0 1 0"/>
     </joint>
    <!--Camera Addtion-->
