Commit message: done urdf

File: rover/src/kipp_description/urdf/kipp.urdf.xacro (robot description, xacro)
@@ -6,15 +6,22 @@
 <xacro:property name="base_height" value="0.51"/>
 <xacro:property name="base_length" value="0.77975"/>
+<xacro:property name="wheel_radius" value="0.0909"/>
+<xacro:property name="wheel_width" value="0.1016"/>
+<xacro:property name="footprint" value="${-((base_height/2)+(wheel_radius))}"/>
 <xacro:property name="steering_xy" value="0.06155"/>
 <xacro:property name="steering_z" value="0.23"/>
-<xacro:property name="wheel_radius" value="0.0909"/>
-<xacro:property name="wheel_width" value="0.1016"/>
-<xacro:property name="camera_y" value=""/>
-<xacro:property name="camera_z" value=""/>
-<xacro:property name="gnss_x" value=""/>
-<xacro:property name="gnss_y" value=""/>
-<xacro:property name="gnss_z" value=""/>
+<xacro:property name="camera_x" value="0.34"/>
+<xacro:property name="camera_z" value="${0.28+footprint}"/>
+<xacro:property name="gnss_x" value="-0.21"/>
+<xacro:property name="gnss_y" value="0.07"/>
+<xacro:property name="gnss_z" value="${0.60+footprint}"/>
+<xacro:property name="gnss_radius" value="0.03"/>
+<xacro:property name="gnss_width" value="0.02"/>
+<!-- <xacro:property name="imu_x" value=""/>
+<xacro:property name="imu_y" value=""/>
+<xacro:property name="imu_z" value=""/>
+<xacro:property name="imu_radius" value=""/>
+<xacro:property name="imu_width" value=""/> -->
 <xacro:property name="PI" value="3.1415692"/>
-<xacro:property name="footprint" value="${-((base_height/2)+(wheel_radius))}"/>
     <!-- Robot Base -->
    <link name="base_link">
@@ -100,5 +107,5 @@
         <child link="middle_left_wheel_link"/>
         <origin xyz="0 ${(base_width)/2} ${footprint}" rpy="0 0 0"/>
-        <axis xyz="0 1 0"/>
+        <axis xyz="0 0 1"/>
     </joint>
     <!-- Middle Right Wheel -->
@@ -118,41 +125,54 @@
         <child link="middle_right_wheel_link"/>
         <origin xyz="0 ${-(base_width)/2} ${footprint}" rpy="0 0 0"/>
-        <axis xyz="0 1 0"/>
+        <axis xyz="0 0 1"/>
     </joint>
+    <!--Sensors -->
    <!--Camera Addtion-->
-    <xacro:arg name="camera_name"   default="zed2i" />
-    <xacro:arg name="camera_model"  default="zed2i" />
-    <xacro:arg name="use_zed_localization" default="true" />
+   <xacro:arg name="camera_name"   default="zed2i" />
+  <xacro:arg name="camera_model"  default="zed2i" />
+  <xacro:arg name="use_zed_localization" default="true" />
     <xacro:zed_camera name="$(arg camera_name)" model="$(arg camera_model)" />
      <!-- Add the first ZED Camera -->
-    <xacro:if value="$(arg use_zed_localization)">
-        <!-- ZED Localization -> The reference link is '$(arg camera_name)_camera_link' and 'base_link' is a child -->
-        <joint name="$(arg camera_name)_joint" type="fixed">
+      <xacro:if value="$(arg use_zed_localization)">
+    <!-- ZED Localization -> The reference link is '$(arg camera_name)_camera_link' and 'base_link' is a child -->
+    <joint name="$(arg camera_name)_joint" type="fixed">
+      <parent link="base_link"/>
+      <child link="$(arg camera_name)_camera_link"/>
+      <origin xyz="${camera_x} 0.0 ${camera_z}" rpy="0 0 0"/>
+    </joint>
+  </xacro:if>
+  <xacro:unless value="$(arg use_zed_localization)">
+    <!-- NO ZED Localization -> '$(arg camera_name)_camera_link' is a child of 'base_link' -->
+    <joint name="$(arg camera_name)_joint" type="fixed">
+      <parent link="base_link"/>
+      <child link="$(arg camera_name)_camera_link"/>
+      <origin xyz="${camera_x} 0.0 ${camera_z}" rpy="0 0 0"/>
+    </joint>
+  </xacro:unless>
+  <link name="gnss_link">
+        <visual>
+            <origin xyz="0.0 0.0 0.0" rpy="0.0 0.0 0.0"/>
+            <geometry>
+                <cylinder radius="${gnss_radius}" length="${gnss_width}"/>
+            </geometry>
+        </visual>
+   </link>
+    <joint name="gnss_joint" type="fixed">
         <parent link="base_link"/>
-        <child link="$(arg camera_name)_camera_link"/>
-        <origin xyz="${camera_y} ${camera_z}" rpy="0 0 0"/>
-        </joint>
-    </xacro:if>
-    <xacro:unless value="$(arg use_zed_localization)">
-        <!-- NO ZED Localization -> '$(arg camera_name)_camera_link' is a child of 'base_link' -->
-        <joint name="$(arg camera_name)_joint" type="fixed">
+        <child link="gnss_link"/>
+        <origin xyz="${gnss_x} ${gnss_y} ${gnss_z}" rpy="0 0 0"/>
+    </joint>
+    <!-- <link name="imu_link">
+        <visual>
+            <origin xyz="0.0 0.0 0.0" rpy="${Pi/2} 0.0 0.0"/>
+            <geometry>
+                <cylinder radius="${imu_radius}" length="{imu_width}"/>
+            </geometry>
+        </visual>
+    </link>
+    <joint name="imu_joint">
         <parent link="base_link"/>
-        <child link="$(arg camera_name)_camera_link"/>
-        <origin xyz="${camera_y} ${camera_z}" rpy="0 0 0"/>
-        </joint>
-    </xacro:unless>
-<!--GNSS-->
-    <link name="gnss_link">
-            <visual>
-                <origin xyz="0.0 0.0 0.0" rpy="1.57 0.0 0.0"/>
-                <geometry>
-                    <cylinder radius="0.05" length="0.05"/> <!-- GNSS radius?-->
-                </geometry>
-            </visual>
-    </link>
-        <joint name="gnss_joint" type="fixed">
-            <parent link="base_link"/>
-            <child link="gnss_link"/>
-            <origin xyz="${gnss_x} ${gnss_y} ${gnss_z}" rpy="0 0 0"/> <!-- GNSS position -->
-        </joint>
+        <child link="imu_link"/>
+        <origin xyz="${imu_x} ${imu_y} ${imu_z}" rpy="0 0 0"/>
+    </joint> -->
 </robot>

Commit message: fixed urdf with zed

File: rover/src/kipp_description/urdf/kipp.urdf.xacro (robot description, xacro)
@@ -132,5 +132,7 @@
   <xacro:arg name="camera_model"  default="zed2i" />
   <xacro:arg name="use_zed_localization" default="true" />
-    <xacro:zed_camera name="$(arg camera_name)" model="$(arg camera_model)" />
+    <xacro:zed_camera name="$(arg camera_name)" model="$(arg camera_model)" enable_gnss="false" custom_baseline="0">
+        <origin xyz="0.0 0.0 0.0" rpy="0 0 0"/>
+    </xacro:zed_camera>
      <!-- Add the first ZED Camera -->
       <xacro:if value="$(arg use_zed_localization)">

Commit message: started robot localization

File: rover/src/kipp_description/urdf/kipp.urdf.xacro (robot description, xacro)
@@ -18,9 +18,9 @@
 <xacro:property name="gnss_radius" value="0.03"/>
 <xacro:property name="gnss_width" value="0.02"/>
-<!-- <xacro:property name="imu_x" value=""/>
-<xacro:property name="imu_y" value=""/>
-<xacro:property name="imu_z" value=""/>
-<xacro:property name="imu_radius" value=""/>
-<xacro:property name="imu_width" value=""/> -->
+<xacro:property name="imu_x" value="-0.21"/>
+<xacro:property name="imu_y" value="0.07"/>
+<xacro:property name="imu_z" value="${0.60+footprint}"/>
+<xacro:property name="imu_radius" value="0.03"/>
+<xacro:property name="imu_width" value="0.02"/>
 <xacro:property name="PI" value="3.1415692"/>
     <!-- Robot Base -->
@@ -165,16 +165,16 @@
         <origin xyz="${gnss_x} ${gnss_y} ${gnss_z}" rpy="0 0 0"/>
     </joint>
-    <!-- <link name="imu_link">
+    <link name="imu_link">
         <visual>
-            <origin xyz="0.0 0.0 0.0" rpy="${Pi/2} 0.0 0.0"/>
+            <origin xyz="0.0 0.0 0.0" rpy="${PI/2} 0.0 0.0"/>
             <geometry>
-                <cylinder radius="${imu_radius}" length="{imu_width}"/>
+                <cylinder radius="${imu_radius}" length="${imu_width}"/>
             </geometry>
         </visual>
     </link>
-    <joint name="imu_joint">
+    <joint name="imu_joint" type="fixed">
         <parent link="base_link"/>
         <child link="imu_link"/>
         <origin xyz="${imu_x} ${imu_y} ${imu_z}" rpy="0 0 0"/>
-    </joint> -->
+    </joint>
 </robot>

Commit message: Commiting from Jetson

File: rover/src/kipp_description/urdf/kipp.urdf.xacro (robot description, xacro)
@@ -1,5 +1,5 @@
 <?xml version="1.0"?>
 <robot xmlns:xacro="http://www.ros.org/wiki/xacro" name="kipp">
-<xacro:include filename="$(find zed_wrapper)/urdf/zed_macro.urdf.xacro"/>
+<!-- <xacro:include filename="$(find zed_wrapper)/urdf/zed_macro.urdf.xacro"/> -->
 <!-- Robot constants-->
 <xacro:property name="base_width" value= "0.5084"/>
@@ -127,29 +127,5 @@
         <axis xyz="0 0 1"/>
     </joint>
-    <!--Sensors -->
-   <!--Camera Addtion-->
-   <xacro:arg name="camera_name"   default="zed2i" />
-  <xacro:arg name="camera_model"  default="zed2i" />
-  <xacro:arg name="use_zed_localization" default="true" />
-    <xacro:zed_camera name="$(arg camera_name)" model="$(arg camera_model)" enable_gnss="true" custom_baseline="0">
-        <origin xyz="0.0 0.0 0.0" rpy="0 0 0"/>
-    </xacro:zed_camera>
-     <!-- Add the first ZED Camera -->
-      <xacro:if value="$(arg use_zed_localization)">
-    <!-- ZED Localization -> The reference link is '$(arg camera_name)_camera_link' and 'base_link' is a child -->
-    <joint name="$(arg camera_name)_joint" type="fixed">
-      <parent link="base_link"/>
-      <child link="$(arg camera_name)_camera_link"/>
-      <origin xyz="${camera_x} 0.0 ${camera_z}" rpy="0 0 0"/>
-    </joint>
-  </xacro:if>
-  <xacro:unless value="$(arg use_zed_localization)">
-    <!-- NO ZED Localization -> '$(arg camera_name)_camera_link' is a child of 'base_link' -->
-    <joint name="$(arg camera_name)_joint" type="fixed">
-      <parent link="base_link"/>
-      <child link="$(arg camera_name)_camera_link"/>
-      <origin xyz="${camera_x} 0.0 ${camera_z}" rpy="0 0 0"/>
-    </joint>
-  </xacro:unless>
+    <!-- Sensors -->
   <link name="gnss_link">
         <visual>

Commit message: ZED URDF WOrking

File: rover/src/kipp_description/urdf/kipp.urdf.xacro (robot description, xacro)
@@ -154,3 +154,34 @@
         <origin xyz="${imu_x} ${imu_y} ${imu_z}" rpy="0 0 0"/>
     </joint>
+    <xacro:arg name="camera_name"   default="zed" />
+    <xacro:arg name="camera_model"  default="zed2i" />
+    <xacro:arg name="use_zed_localization" default="true" />
+    <!-- ZED DOCUMENTATION OUT OF DATE AS OF FEB 25 2025, must add orgin -->
+    <xacro:include filename="$(find zed_wrapper)/urdf/zed_macro.urdf.xacro" />
+    <xacro:zed_camera name="$(arg camera_name)" model="$(arg camera_model)" enable_gnss="true">
+            <origin xyz="-0.12 0.0 -0.25" rpy="0 0 0"/>
+    </xacro:zed_camera>
+      <!-- Add a joint to connect the ZED Camera to the robot -->
+    <xacro:if value="$(arg use_zed_localization)">
+        <!-- ZED Localization -> The reference link is '$(arg camera_name)_camera_link' and 'base_link' is a child -->
+        <joint name="$(arg camera_name)_joint" type="fixed">
+        <parent link="$(arg camera_name)_camera_link"/>
+        <child link="base_link"/>
+        <origin
+            xyz="-0.12 0.0 -0.25"
+            rpy="0 0 0"
+        />
+        </joint>
+    </xacro:if>
+    <xacro:unless value="$(arg use_zed_localization)">
+        <!-- NO ZED Localization -> '$(arg camera_name)_camera_link' is a child of 'base_link' -->
+        <joint name="$(arg camera_name)_joint" type="fixed">
+        <parent link="base_link"/>
+        <child link="$(arg camera_name)_camera_link"/>
+        <origin
+            xyz="0.12 0.0 0.25"
+            rpy="0 0 0"
+        />
+        </joint>
+    </xacro:unless>
 </robot>

Commit message: Changed Nomapsyaml to reflect rover

File: rover/src/kipp_description/urdf/kipp.urdf.xacro (robot description, xacro)
@@ -23,4 +23,5 @@
 <xacro:property name="imu_radius" value="0.03"/>
 <xacro:property name="imu_width" value="0.02"/>
+<xacro:property name="height_offset" value="0.1"/>
 <xacro:property name="PI" value="3.1415692"/>
     <!-- Robot Base -->

Commit message: gazebo world

File: rover/src/kipp_description/urdf/kipp.urdf.xacro (robot description, xacro)
@@ -1,5 +1,4 @@
 <?xml version="1.0"?>
 <robot xmlns:xacro="http://www.ros.org/wiki/xacro" name="kipp">
-<!-- <xacro:include filename="$(find zed_wrapper)/urdf/zed_macro.urdf.xacro"/> -->
 <!-- Robot constants-->
 <xacro:property name="base_width" value= "0.5084"/>
@@ -11,6 +10,4 @@
 <xacro:property name="steering_xy" value="0.06155"/>
 <xacro:property name="steering_z" value="0.23"/>
-<xacro:property name="camera_x" value="0.34"/>
-<xacro:property name="camera_z" value="${0.28+footprint}"/>
 <xacro:property name="gnss_x" value="-0.21"/>
 <xacro:property name="gnss_y" value="0.07"/>
@@ -155,34 +152,3 @@
         <origin xyz="${imu_x} ${imu_y} ${imu_z}" rpy="0 0 0"/>
     </joint>
-    <xacro:arg name="camera_name"   default="zed" />
-    <xacro:arg name="camera_model"  default="zed2i" />
-    <xacro:arg name="use_zed_localization" default="true" />
-    <!-- ZED DOCUMENTATION OUT OF DATE AS OF FEB 25 2025, must add orgin -->
-    <xacro:include filename="$(find zed_wrapper)/urdf/zed_macro.urdf.xacro" />
-    <xacro:zed_camera name="$(arg camera_name)" model="$(arg camera_model)" enable_gnss="true">
-            <origin xyz="-0.12 0.0 -0.25" rpy="0 0 0"/>
-    </xacro:zed_camera>
-      <!-- Add a joint to connect the ZED Camera to the robot -->
-    <xacro:if value="$(arg use_zed_localization)">
-        <!-- ZED Localization -> The reference link is '$(arg camera_name)_camera_link' and 'base_link' is a child -->
-        <joint name="$(arg camera_name)_joint" type="fixed">
-        <parent link="$(arg camera_name)_camera_link"/>
-        <child link="base_link"/>
-        <origin
-            xyz="-${camera_x} 0 ${camera_z}"
-            rpy="0 0 0"
-        />
-        </joint>
-    </xacro:if>
-    <xacro:unless value="$(arg use_zed_localization)">
-        <!-- NO ZED Localization -> '$(arg camera_name)_camera_link' is a child of 'base_link' -->
-        <joint name="$(arg camera_name)_joint" type="fixed">
-        <parent link="base_link"/>
-        <child link="$(arg camera_name)_camera_link"/>
-        <origin
-            xyz="0.12 0.0 0.25"
-            rpy="0 0 0"
-        />
-        </joint>
-    </xacro:unless>
 </robot>
